Commit message: scales of stl-s are corrected and properly displayed

File: study_description/urdf/manipulator.urdf (robot description, URDF)
Before this commit: robot study_manipulator, 5 links, 4 joints
Joints:
- joint ee: origin xyz=0.2  0 0 rpy=0 0 0 -> xyz=0 0.2 0 rpy=0 0 0
- joint joint1: origin xyz=0 0 1 rpy=0 0 0 -> xyz=0 0 0.1 rpy=0 0 0
- joint joint2: origin xyz=0. 0 5 rpy=0 0 0 -> xyz=0. 0 0.5 rpy=1.5707963267948966 0 0
- joint joint3: origin xyz=0.5 0. -0. rpy=0 0 0 -> xyz=0 0.5 -0. rpy=0 0 0
